File: PCB/Leaf-PAR/Leaf-PAR.kicad_pcb (KiCad board)
At the start: 4 copper layers, 38 x 22.5 mm, 17 parts, among them T1 PPTC081LFBN-RC, U1 AZ1117CR-3.3TRG1, U2 OPA388IDBVT, U3 SN74LV4051ARGYR

Commit message: KiCAD 8
Projected updated to KiCAD 8
Other:
- net class Default removed
